File: hardware/main-board/3117_AUSIGN.kicad_sch (KiCad schematic)
At the start: 151 parts, among them J1 JST_PH_2P, J10 Conn_01x04_Pin, J11 Conn_01x04_Socket, J12 Conn_01x02_Pin, J2 JST_SH_4P, J3 USB4105-GF-A, J4 JST_SH_2P, J5 JST_SH_2P, J6 JST_SH_2P, J7 JST_SH_2P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

Commit message: cleaned up schematic
Other:
- note added: "MISC"
- note added: "Power Supply Subsystem"
- note added: "Processing Subsystem"
- note added: "Sensor Subsystem"
- note added: "User Interface Subsystem"
- note added: "mounting holes"
- note added: "noted errors: C & E on Q3 should be connected in reverse and its layout must also be changed"
- note removed: "MCU"
- note removed: "Peripherals"
- note removed: "Power Supply + USB"
- note removed: "Sensors"
- note removed: "check if we need interupts"
- moved on the sheet: C10, C12, C13, C14, C15, C18, C22, C26, C27, C28, C3, C30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
